File: waddle.kicad_pcb (KiCad board)
At the start: 4 copper layers, 97.7 x 65 mm, 144 parts, among them J1 PJ-102A, J2 USB, J3 TEST_IO, J4 DA PROG, J5 DA PROG, J6 Conn_Coaxial, J7 Power, J8 LED_OUT, J9 PWM_SELECT, SW1 STM_RESET, U1 TPS2065C, U2 STM32F405RGT6, U3 DA14531-00, U4 TPS5430, U5 TPS5430, U6 LSM6DSLTR, Y1 32.768KHz, Y2 32MHZ, Y3 8MHz

Commit message: Update waddle.kicad_pcb
Parts:
- moved C20 3.23 mm to (107.7, 88.2)
- moved C28 3.23 mm to (107.7, 95.8)
- moved D19 3.23 mm to (111.4, 73.5)
- moved D20 3.23 mm to (111.4, 88.2)
- moved D28 3.23 mm to (111.4, 95.8)
- moved C22 3.23 mm to (115.1, 88.2)
- moved C24 3.23 mm to (122.5, 88.2)
- moved C26 3.23 mm to (129.9, 88.2)
- moved C30 3.23 mm to (115.1, 95.8)
- moved C32 3.23 mm to (122.5, 95.8)
- moved D21 3.23 mm to (118.8, 73.5)
- moved D22 3.23 mm to (118.8, 88.2)
- moved D23 3.23 mm to (126.3, 73.5)
- moved D24 3.23 mm to (126.3, 88.2)
- moved D25 3.23 mm to (133.7, 73.5)
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Routing:
- net Net-(D34-DOUT): track 38.1 -> 40.0 mm
- net Net-(D19-DIN): track 41.8 -> 40.0 mm
- net /test_points/TP06: track 57.9 -> 56.2 mm
- net /test_points/TP05: track 61.1 -> 60.1 mm
- net /power/+5V: track 293.4 -> 292.6 mm
